File: _autosave-laser.kicad_sch (KiCad schematic)
At the start: 14 parts, among them J1 Conn_Coaxial, J2 Conn_02x06, J3 Conn_Coaxial, Q1 BS170, Q2 BS170

Commit message: insert C
Parts:
- added C3: 10u, Capacitor_THT:CP_Radial_D5.0mm_P2.50mm, symbol Device:C_Polarized
- added C4: 100n, Capacitor_THT:C_Rect_L7.0mm_W6.0mm_P5.00mm, symbol Device:C
Connections:
- net +3.3V: now also C3.1, C4.1
- net GND: now also C3.2, C4.2
Changed lines of the file:
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@@
   (junction (at 198.12 139.7) (diameter 0) (color 0 0 0 0)
   )
+  (junction (at 190.5 73.66) (diameter 0) (color 0 0 0 0)
+  )
   (junction (at 138.43 110.49) (diameter 0) (color 0 0 0 0)
   )
+  (junction (at 199.39 53.34) (diameter 0) (color 0 0 0 0)
+  )
   (junction (at 138.43 134.62) (diameter 0) (color 0 0 0 0)
   )
@@
     (stroke (width 0) (type default))
   )
+  (wire (pts (xy 190.5 58.42) (xy 190.5 53.34))
+    (stroke (width 0) (type default))
+  )
+  (wire (pts (xy 199.39 66.04) (xy 199.39 73.66))
+    (stroke (width 0) (type default))
+  )
   (wire (pts (xy 138.43 105.41) (xy 138.43 110.49))
     (stroke (width 0) (type default))
   )
+  (wire (pts (xy 190.5 73.66) (xy 190.5 74.93))
+    (stroke (width 0) (type default))
+  )
   (wire (pts (xy 148.59 58.42) (xy 148.59 53.34))
     (stroke (width 0) (type default))
@@
     (stroke (width 0) (type default))
   )
+  (wire (pts (xy 199.39 53.34) (xy 199.39 58.42))
+    (stroke (width 0) (type default))
+  )
+  (wire (pts (xy 199.39 50.8) (xy 199.39 53.34))
+    (stroke (width 0) (type default))
+  )
   (wire (pts (xy 198.12 115.57) (xy 209.55 115.57))
     (stroke (width 0) (type default))
@@
     (stroke (width 0) (type default))
   )
+  (wire (pts (xy 190.5 73.66) (xy 199.39 73.66))
+    (stroke (width 0) (type default))
+  )
   (wire (pts (xy 118.11 64.77) (xy 120.65 64.77))
     (stroke (width 0) (type default))
@@
     (stroke (width 0) (type default))
   )
+  (wire (pts (xy 190.5 53.34) (xy 199.39 53.34))
+    (stroke (width 0) (type default))
+  )
   (wire (pts (xy 138.43 110.49) (xy 138.43 111.76))
     (stroke (width 0) (type default))
@@
   )
   (wire (pts (xy 127 130.81) (xy 127 134.62))
+    (stroke (width 0) (type default))
+  )
+  (wire (pts (xy 190.5 66.04) (xy 190.5 73.66))
     (stroke (width 0) (type default))
   )
@@
         (path "/36036e48-7fe7-4c15-b22f-192311846a69"
           (reference "Q1") (unit 1)
+        )
+      )
+    )
+  )
+  (symbol (lib_id "Device:C_Polarized") (at 190.5 62.23 0) (unit 1)
+    (in_bom yes) (on_board yes) (dnp no)
+    (property "Reference" "C3" (at 185.42 57.15 0)
+      (effects (font (size 1.27 1.27)) (justify left))
+    )
+    (property "Value" "10u" (at 185.42 66.04 0)
+      (effects (font (size 1.27 1.27)) (justify left))
+    )
+    (property "Footprint" "Capacitor_THT:CP_Radial_D5.0mm_P2.50mm" (at 191.4652 66.04 0)
+      (effects (font (size 1.27 1.27)) hide)
+    )
+    (property "Datasheet" "~" (at 190.5 62.23 0)
+      (effects (font (size 1.27 1.27)) hide)
+    )
+    (pin "1")
+    (pin "2")
+    (instances
+      (project "laser"
+        (path "/36036e48-7fe7-4c15-b22f-192311846a69"
+          (reference "C3") (unit 1)
         )
       )
@@
     )
   )
+  (symbol (lib_id "power:GND") (at 190.5 74.93 0) (unit 1)
+    (in_bom yes) (on_board yes) (dnp no) (fields_autoplaced)
+    (property "Reference" "#PWR017" (at 190.5 81.28 0)
+      (effects (font (size 1.27 1.27)) hide)
+    )
+    (property "Value" "GND" (at 190.5 80.01 0)
+      (effects (font (size 1.27 1.27)))
+    )
+    (property "Footprint" "" (at 190.5 74.93 0)
+      (effects (font (size 1.27 1.27)) hide)
+    )
+    (property "Datasheet" "" (at 190.5 74.93 0)
+      (effects (font (size 1.27 1.27)) hide)
+    )
+    (pin "1")
+    (instances
+      (project "laser"
+        (path "/36036e48-7fe7-4c15-b22f-192311846a69"
+          (reference "#PWR017") (unit 1)
+        )
+      )
+    )
+  )
   (symbol (lib_id "power:+3.3V") (at 116.84 104.14 270) (unit 1)
     (in_bom yes) (on_board yes) (dnp no) (fields_autoplaced)
@@
     )
   )
+  (symbol (lib_id "power:+3.3V") (at 199.39 50.8 0) (unit 1)
+    (in_bom yes) (on_board yes) (dnp no) (fields_autoplaced)
+    (property "Reference" "#PWR018" (at 199.39 54.61 0)
+      (effects (font (size 1.27 1.27)) hide)
+    )
+    (property "Value" "+3.3V" (at 199.39 46.99 0)
+      (effects (font (size 1.27 1.27)))
+    )
+    (property "Footprint" "" (at 199.39 50.8 0)
+      (effects (font (size 1.27 1.27)) hide)
+    )
+    (property "Datasheet" "" (at 199.39 50.8 0)
+      (effects (font (size 1.27 1.27)) hide)
+    )
+    (pin "1")
+    (instances
+      (project "laser"
+        (path "/36036e48-7fe7-4c15-b22f-192311846a69"
+          (reference "#PWR018") (unit 1)
+        )
+      )
+    )
+  )
   (symbol (lib_id "power:+5V") (at 138.43 95.25 0) (unit 1)
     (in_bom yes) (on_board yes) (dnp no) (fields_autoplaced)
@@
         )
       )
+    )
+  )
+  (symbol (lib_id "Device:C") (at 199.39 62.23 0) (unit 1)
+    (in_bom yes) (on_board yes) (dnp no)
+    (property "Reference" "C4" (at 195.58 57.15 0)
+      (effects (font (size 1.27 1.27)) (justify left))
+    )
+    (property "Value" "100n" (at 194.31 66.04 0)
+      (effects (font (size 1.27 1.27)) (justify left))
+    )
+    (property "Footprint" "Capacitor_THT:C_Rect_L7.0mm_W6.0mm_P5.00mm" (at 200.3552 66.04 0)
+      (effects (font (size 1.27 1.27)) hide)
+    )
+    (property "Datasheet" "~" (at 199.39 62.23 0)
+      (effects (font (size 1.27 1.27)) hide)
+    )
+    (pin "1")
+    (pin "2")
+    (instances
+      (project "laser"
+        (path "/36036e48-7fe7-4c15-b22f-192311846a69"
+          (reference "C4") (unit 1)
+        )
+      )
