File: laser.kicad_pcb (KiCad board)
At the start: 2 copper layers, 50 x 50 mm, 16 parts, among them J1 Conn_Coaxial, J2 Conn_02x06, J3 Conn_Coaxial, Q1 BS170, Q2 BS170

Commit message: insert C
Parts:
- removed the ? at (147.3, 116.5)
- removed the ? at (163.5, 116.5)
- added ?: , , F.Cu at (167.3, 116.1)
- added ?: , , F.Cu at (158.6, 116.1)
- added C3: 10u, Capacitor_THT:CP_Radial_D5.0mm_P2.50mm, F.Cu at (131.9, 113.3)
- added C4: 100n, Capacitor_THT:C_Rect_L7.0mm_W6.0mm_P5.00mm, F.Cu at (131.9, 118.1)
- moved U1 7.28 mm to (137.9, 110.5)
- moved J2 6.08 mm to (163.6, 119.6)
- moved R2 6.01 mm to (167.5, 112.0)
- moved Q1 1.36 mm to (138.1, 95.4)
- moved Q2 0.59 mm to (170.2, 106.2)
Routing:
- net +3.3V: track 16.5 -> 26.2 mm
- net GND: track 16.2 -> 8.70 mm
- net Net-(J2-Pin_1): track 93.4 -> 90.0 mm
- net LaserIn: track 37.3 -> 34.5 mm
- net Net-(J1-In): track 40.2 -> 38.5 mm
- net Net-(J3-In): track 22.1 -> 22.8 mm
Other:
- board text added: "https://github.com/Johann-Schmid/laser"

Commit message: change the bnc connector of the backplane
change the bnc connector of the backplane
Parts:
- J1, J3: moved to B.Cu
- turned J1 to 180 degrees
- turned J3 to 180 degrees

Commit message: mounting hole
Parts:
- added REF**: MountingHole_4.3mm_M4, MountingHole:MountingHole_4.3mm_M4, F.Cu at (152.5, 87.7)
- R3: moved to B.Cu
Changed lines of the file:
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@@
-  )
-  (footprint "Resistor_THT:R_Axial_DIN0411_L9.9mm_D3.6mm_P20.32mm_Horizontal" (layer "F.Cu")
-    (at 145.796 99.06 90)
-    (descr "Resistor, Axial_DIN0411 series, Axial, Horizontal, pin pitch=20.32mm, 1W, length*diameter=9.9*3.6mm^2")
-    (tags "Resistor Axial_DIN0411 series Axial Horizontal pin pitch 20.32mm 1W length 9.9mm diameter 3.6mm")
-    (property "Sheetfile" "laser.kicad_sch")
-    (property "Sheetname" "")
-    (property "ki_description" "Resistor")
-    (property "ki_keywords" "R res resistor")
-    (attr through_hole)
-    (fp_text reference "R3" (at 10.16 -2.92 90) (layer "F.SilkS")
-        (effects (font (size 1 1) (thickness 0.15)))
-    )
-    (fp_text value "1.5k" (at 10.16 2.92 90) (layer "F.Fab")
-        (effects (font (size 1 1) (thickness 0.15)))
-    )
-    (fp_text user "${REFERENCE}" (at 10.16 0 90) (layer "F.Fab")
-        (effects (font (size 1 1) (thickness 0.15)))
-    )
-    (fp_line (start 1.44 0) (end 5.09 0)
-      (stroke (width 0.12) (type solid)) (layer "F.SilkS"))
-    (fp_line (start 5.09 -1.92) (end 5.09 1.92)
-      (stroke (width 0.12) (type solid)) (layer "F.SilkS"))
-    (fp_line (start 5.09 1.92) (end 15.23 1.92)
-      (stroke (width 0.12) (type solid)) (layer "F.SilkS"))
-    (fp_line (start 15.23 -1.92) (end 5.09 -1.92)
-      (stroke (width 0.12) (type solid)) (layer "F.SilkS"))
-    (fp_line (start 15.23 1.92) (end 15.23 -1.92)
-      (stroke (width 0.12) (type solid)) (layer "F.SilkS"))
-    (fp_line (start 18.88 0) (end 15.23 0)
-      (stroke (width 0.12) (type solid)) (layer "F.SilkS"))
-    (fp_line (start -1.45 -2.05) (end -1.45 2.05)
-      (stroke (width 0.05) (type solid)) (layer "F.CrtYd"))
-    (fp_line (start -1.45 2.05) (end 21.77 2.05)
-      (stroke (width 0.05) (type solid)) (layer "F.CrtYd"))
-    (fp_line (start 21.77 -2.05) (end -1.45 -2.05)
-      (stroke (width 0.05) (type solid)) (layer "F.CrtYd"))
-    (fp_line (start 21.77 2.05) (end 21.77 -2.05)
-      (stroke (width 0.05) (type solid)) (layer "F.CrtYd"))
-    (fp_line (start 0 0) (end 5.21 0)
-      (stroke (width 0.1) (type solid)) (layer "F.Fab"))
-    (fp_line (start 5.21 -1.8) (end 5.21 1.8)
-      (stroke (width 0.1) (type solid)) (layer "F.Fab"))
-    (fp_line (start 5.21 1.8) (end 15.11 1.8)
-      (stroke (width 0.1) (type solid)) (layer "F.Fab"))
-    (fp_line (start 15.11 -1.8) (end 5.21 -1.8)
-      (stroke (width 0.1) (type solid)) (layer "F.Fab"))
-    (fp_line (start 15.11 1.8) (end 15.11 -1.8)
-      (stroke (width 0.1) (type solid)) (layer "F.Fab"))
-    (fp_line (start 20.32 0) (end 15.11 0)
-      (stroke (width 0.1) (type solid)) (layer "F.Fab"))
-    (pad "1" thru_hole circle (at 0 0 90) (size 2.4 2.4) (drill 1.2) (layers "*.Cu" "*.Mask")
-      (net 1 "+5V") (pintype "passive"))
-    (pad "2" thru_hole oval (at 20.32 0 90) (size 2.4 2.4) (drill 1.2) (layers "*.Cu" "*.Mask")
-      (net 3 "Net-(D1-A)") (pintype "passive"))
-    (model "${KICAD6_3DMODEL_DIR}/Resistor_THT.3dshapes/R_Axial_DIN0411_L9.9mm_D3.6mm_P20.32mm_Horizontal.wrl"
-      (offset (xyz 0 0 0))
-      (scale (xyz 1 1 1))
-      (rotate (xyz 0 0 0))
-    )
   )
   (footprint "Resistor_THT:R_Axial_DIN0411_L9.9mm_D3.6mm_P20.32mm_Horizontal" (layer "F.Cu")
@@
     )
   )
+  (footprint "MountingHole:MountingHole_4.3mm_M4" (layer "F.Cu")
+    (at 152.52 87.68)
+    (descr "Mounting Hole 4.3mm, no annular, M4")
+    (tags "mounting hole 4.3mm no annular m4")
+    (attr exclude_from_pos_files exclude_from_bom)
+    (fp_text reference "REF**" (at 0 -5.3) (layer "F.SilkS")
+        (effects (font (size 1 1) (thickness 0.15)))
+    )
+    (fp_text value "MountingHole_4.3mm_M4" (at 0 5.3) (layer "F.Fab")
+        (effects (font (size 1 1) (thickness 0.15)))
+    )
+    (fp_text user "${REFERENCE}" (at 0 0) (layer "F.Fab")
+        (effects (font (size 1 1) (thickness 0.15)))
+    )
+    (fp_circle (center 0 0) (end 4.3 0)
+      (stroke (width 0.15) (type solid)) (fill none) (layer "Cmts.User"))
+    (fp_circle (center 0 0) (end 4.55 0)
+      (stroke (width 0.05) (type solid)) (fill none) (layer "F.CrtYd"))
+    (pad "" np_thru_hole circle (at 0 0) (size 4.3 4.3) (drill 4.3) (layers "*.Cu" "*.Mask"))
+  )
   (footprint "Resistor_THT:R_Axial_DIN0411_L9.9mm_D3.6mm_P20.32mm_Horizontal" (layer "F.Cu")
     (at 150.368 100.076)
@@
       (offset (xyz 0 0 0))
       (scale (xyz 1 1 1))
+      (rotate (xyz 0 0 0))
+    )
+  )
+  (footprint "Resistor_THT:R_Axial_DIN0411_L9.9mm_D3.6mm_P20.32mm_Horizontal" (layer "B.Cu")
+    (at 145.796 99.06 90)
+    (descr "Resistor, Axial_DIN0411 series, Axial, Horizontal, pin pitch=20.32mm, 1W, length*diameter=9.9*3.6mm^2")
+    (tags "Resistor Axial_DIN0411 series Axial Horizontal pin pitch 20.32mm 1W length 9.9mm diameter 3.6mm")
+    (property "Sheetfile" "laser.kicad_sch")
+    (property "Sheetname" "")
+    (property "ki_description" "Resistor")
+    (property "ki_keywords" "R res resistor")
+    (attr through_hole)
+    (fp_text reference "R3" (at 10.16 2.92 90) (layer "B.SilkS")
+        (effects (font (size 1 1) (thickness 0.15)) (justify mirror))
+    )
+    (fp_text value "1.5k" (at 10.16 -2.92 90) (layer "B.Fab")
+        (effects (font (size 1 1) (thickness 0.15)) (justify mirror))
+    )
+    (fp_text user "${REFERENCE}" (at 10.16 0 90) (layer "B.Fab")
+        (effects (font (size 1 1) (thickness 0.15)) (justify mirror))
+    )
+    (fp_line (start 1.44 0) (end 5.09 0)
+      (stroke (width 0.12) (type solid)) (layer "B.SilkS"))
+    (fp_line (start 5.09 -1.92) (end 15.23 -1.92)
+      (stroke (width 0.12) (type solid)) (layer "B.SilkS"))
+    (fp_line (start 5.09 1.92) (end 5.09 -1.92)
+      (stroke (width 0.12) (type solid)) (layer "B.SilkS"))
+    (fp_line (start 15.23 -1.92) (end 15.23 1.92)
+      (stroke (width 0.12) (type solid)) (layer "B.SilkS"))
+    (fp_line (start 15.23 1.92) (end 5.09 1.92)
+      (stroke (width 0.12) (type solid)) (layer "B.SilkS"))
+    (fp_line (start 18.88 0) (end 15.23 0)
+      (stroke (width 0.12) (type solid)) (layer "B.SilkS"))
+    (fp_line (start -1.45 -2.05) (end 21.77 -2.05)
+      (stroke (width 0.05) (type solid)) (layer "B.CrtYd"))
+    (fp_line (start -1.45 2.05) (end -1.45 -2.05)
+      (stroke (width 0.05) (type solid)) (layer "B.CrtYd"))
+    (fp_line (start 21.77 -2.05) (end 21.77 2.05)
+      (stroke (width 0.05) (type solid)) (layer "B.CrtYd"))
+    (fp_line (start 21.77 2.05) (end -1.45 2.05)
+      (stroke (width 0.05) (type solid)) (layer "B.CrtYd"))
+    (fp_line (start 0 0) (end 5.21 0)
+      (stroke (width 0.1) (type solid)) (layer "B.Fab"))
+    (fp_line (start 5.21 -1.8) (end 15.11 -1.8)
+      (stroke (width 0.1) (type solid)) (layer "B.Fab"))
+    (fp_line (start 5.21 1.8) (end 5.21 -1.8)
+      (stroke (width 0.1) (type solid)) (layer "B.Fab"))
+    (fp_line (start 15.11 -1.8) (end 15.11 1.8)
+      (stroke (width 0.1) (type solid)) (layer "B.Fab"))
+    (fp_line (start 15.11 1.8) (end 5.21 1.8)
+      (stroke (width 0.1) (type solid)) (layer "B.Fab"))
+    (fp_line (start 20.32 0) (end 15.11 0)
+      (stroke (width 0.1) (type solid)) (layer "B.Fab"))
+    (pad "1" thru_hole circle (at 0 0 90) (size 2.4 2.4) (drill 1.2) (layers "*.Cu" "*.Mask")
+      (net 1 "+5V") (pintype "passive"))
+    (pad "2" thru_hole oval (at 20.32 0 90) (size 2.4 2.4) (drill 1.2) (layers "*.Cu" "*.Mask")
+      (net 3 "Net-(D1-A)") (pintype "passive"))
+    (model "${KICAD6_3DMODEL_DIR}/Resistor_THT.3dshapes/R_Axial_DIN0411_L9.9mm_D3.6mm_P20.32mm_Horizontal.wrl"
+      (offset (xyz 0 0 0))
+      (scale (xyz 1 1 1))
